File: guitar-effect.kicad_sch (KiCad schematic)
At the start: 34 parts, among them IC1 PCM3002E, J1 Conn_01x07_Pin, J2 Conn_01x07_Pin, U1 MCP6004, U2 MCP6004

Commit message: Add files via upload
Voltage regulators
Parts:
- added C19, C23, C24, C4: 10u, Capacitor_SMD:C_0805_2012Metric, symbol Device:C
- added C20, C21, C26, C27: 22u, Capacitor_SMD:C_0805_2012Metric, symbol Device:C
- added C22, C25: 100n, Capacitor_SMD:C_0805_2012Metric, symbol Device:C
- added IC2, IC3: TPS563209DDCR, SamacSys_Parts:SOT95P280X110-6N, symbol SamacSys_Parts:TPS563209DDCR
- added L1, L2: 4.7u, symbol Device:L
- added R12: 20k, Resistor_SMD:R_0805_2012Metric, symbol Device:R
- added R13: 3.6k, Resistor_SMD:R_0805_2012Metric, symbol Device:R
- added R14: 3.3k, Resistor_SMD:R_0805_2012Metric, symbol Device:R
- added R15: 1k, Resistor_SMD:R_0805_2012Metric, symbol Device:R
- C1, C14, C15, C16, C2, C3, C9: footprint (none) -> Capacitor_SMD:C_0805_2012Metric
- C_Polarized1: renamed from 0.1u; value C_Polarized -> 0.1u; footprint (none) -> Capacitor_SMD:CP_Elec_8x5.4
- C_Polarized10: renamed from C10; footprint (none) -> Capacitor_SMD:CP_Elec_8x5.4
- C_Polarized11: renamed from C11; footprint (none) -> Capacitor_SMD:CP_Elec_8x5.4
- C_Polarized2: renamed from C18; footprint (none) -> Capacitor_SMD:CP_Elec_8x5.4
- C_Polarized3: renamed from C6; footprint (none) -> Capacitor_SMD:CP_Elec_8x5.4
- C_Polarized4: renamed from C17; footprint (none) -> Capacitor_SMD:CP_Elec_8x5.4
- C_Polarized5: renamed from C12; footprint (none) -> Capacitor_SMD:CP_Elec_8x5.4
- C_Polarized6: renamed from C13; footprint (none) -> Capacitor_SMD:CP_Elec_8x5.4
- C_Polarized7: renamed from C7; footprint (none) -> Capacitor_SMD:CP_Elec_8x5.4
- C_Polarized8: renamed from C8; footprint (none) -> Capacitor_SMD:CP_Elec_8x5.4
- C_Polarized9: renamed from C5; footprint (none) -> Capacitor_SMD:CP_Elec_8x5.4
- IC1: footprint SOP65P780X200-24N -> SamacSys_Parts:SOP65P780X200-24N
- R1, R10, R11, R2, R3, R4, R5, R6, R7, R8, R9: footprint (none) -> Resistor_SMD:R_0805_2012Metric
Connections:
- net VCC renamed +3V3
- net +3V3: now also C26.1, C27.1, L2.2, R14.1; no longer U2.4 (V+)
- new net: IC3.4 (VFB), R14.2, R15.1
- new net: IC2.4 (VFB), R12.2, R13.1
- new net: C25.1, IC3.2 (SW)
- new net: C25.2, IC3.6 (VBST), L2.1
- new net: C22.2, IC2.6 (VBST), L1.1
- new net: C22.1, IC2.2 (SW)
- new net +12V: C19.1, C23.1, C24.1, C4.1, IC2.3 (VIN), IC2.5 (EN), IC3.3 (VIN), IC3.5 (EN)
- new net +5VD: C20.1, C21.1, L1.2, R12.1, U2.4 (V+)
- new net GND: C19.2, C20.2, C21.2, C23.2, C24.2, C26.2, C27.2, C4.2, IC2.1 (GND), IC3.1 (GND), R13.2, R15.2
Other:
- moved on the sheet: C1, C14, C15, C16, C2, C3, J1, J2, R1, R10, R11, R2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

Commit message: PCB design
Power supply withs LDOs added to schematic. V1.0 PCB design. Gerber and drill files
Parts:
- removed C19, C23, C24: 10u, Capacitor_SMD:C_0805_2012Metric, symbol Device:C
- removed C20, C21, C26, C27: 22u, Capacitor_SMD:C_0805_2012Metric, symbol Device:C
- removed C22: 100n, Capacitor_SMD:C_0805_2012Metric, symbol Device:C
- removed C9: 0.1u, Capacitor_SMD:C_0805_2012Metric, symbol Device:C
- removed IC2, IC3: TPS563209DDCR, SamacSys_Parts:SOT95P280X110-6N, symbol SamacSys_Parts:TPS563209DDCR
- removed J1, J2: Conn_01x07_Pin, symbol Connector:Conn_01x07_Pin
- removed R12: 20k, Resistor_SMD:R_0805_2012Metric, symbol Device:R
- removed R13: 3.6k, Resistor_SMD:R_0805_2012Metric, symbol Device:R
- removed R14: 3.3k, Resistor_SMD:R_0805_2012Metric, symbol Device:R
- removed R15: 1k, Resistor_SMD:R_0805_2012Metric, symbol Device:R
- removed R6: 10k, Resistor_SMD:R_0805_2012Metric, symbol Device:R
- removed U1, U2: MCP6004, symbol Amplifier_Operational:MCP6004
- added C1, C2, C6: 0.1u, Capacitor_SMD:C_0805_2012Metric, symbol Device:C
- added C3, C5, C7, C8: 100n, Capacitor_SMD:C_0805_2012Metric, symbol Device:C
- added C_Polarized12: 10u, Capacitor_THT:CP_Radial_D4.0mm_P1.50mm, symbol Device:C_Polarized
- added D1, D2: S2BA-13-F, Diode_SMD:D_SMA, symbol Device:D
- added IC4, IC5: MCP6007-E_SN, SamacSys_Parts:SOIC127P600X175-8N, symbol SamacSys_Parts:MCP6007-E_SN
- added J1: Barrel_Jack_Switch, Connector_BarrelJack:BarrelJack_Horizontal, symbol Connector:Barrel_Jack_Switch
- added J2: Conn_01x11_Pin, Connector_PinSocket_2.54mm:PinSocket_1x11_P2.54mm_Vertical, symbol Connector:Conn_01x11_Pin
- added J3: Conn_01x08_Pin, Connector_PinSocket_2.54mm:PinSocket_1x08_P2.54mm_Vertical, symbol Connector:Conn_01x08_Pin
- added J4, J5: NRJ4HF, Connector_Audio:Jack_6.35mm_Neutrik_NRJ4HF_Horizontal, symbol Connector_Audio:NRJ4HF
- added R1, R16, R17: 10k, Resistor_SMD:R_0805_2012Metric, symbol Device:R
- added U1: LD1117S12TR_SOT223, Package_TO_SOT_SMD:SOT-223-3_TabPin2, symbol Regulator_Linear:LD1117S12TR_SOT223
- added U2: LD1117S33TR_SOT223, Package_TO_SOT_SMD:SOT-223-3_TabPin2, symbol Regulator_Linear:LD1117S33TR_SOT223
- C4: value 10u -> 100n
- C_Polarized1: value 0.1u -> 10u; footprint Capacitor_SMD:CP_Elec_8x5.4 -> Capacitor_THT:CP_Radial_D4.0mm_P1.50mm
- C_Polarized10: value 4.7u -> 1u; footprint Capacitor_SMD:CP_Elec_8x5.4 -> Capacitor_THT:CP_Radial_D4.0mm_P1.50mm
- C_Polarized11, C_Polarized2, C_Polarized5, C_Polarized7, C_Polarized9: footprint Capacitor_SMD:CP_Elec_8x5.4 -> Capacitor_THT:CP_Radial_D4.0mm_P1.50mm
- C_Polarized3: value 0.1u -> 4.7u; footprint Capacitor_SMD:CP_Elec_8x5.4 -> Capacitor_THT:CP_Radial_D4.0mm_P1.50mm
- C_Polarized4: value 10u -> 4.7u; footprint Capacitor_SMD:CP_Elec_8x5.4 -> Capacitor_THT:CP_Radial_D4.0mm_P1.50mm
- C_Polarized6: value 1u -> 4.7u; footprint Capacitor_SMD:CP_Elec_8x5.4 -> Capacitor_THT:CP_Radial_D4.0mm_P1.50mm
- C_Polarized8: value 4.7u -> 4.7u Tantalllum; footprint Capacitor_SMD:CP_Elec_8x5.4 -> Capacitor_THT:CP_Radial_D4.0mm_P1.50mm
- L1, L2: value 4.7u -> 10u; footprint (none) -> Inductor_SMD:L_0805_2012Metric_Pad1.15x1.40mm_HandSolder
- renumbered C14 to C11, C3 to C12, C15 to C16, C2 to C17, C16 to C18, C1 to C19, R9 to R10, R2 to R11, R10 to R13, R5 to R14, R8 to R3, R7 to R6, R3 to R7, R11 to R8, R1 to R9
Connections:
- net GND1 is gone; now on net VGND: R13.1, R14.1, R3.2, R4.2
- net BIT: now also J2.2 (Pin_2)
- net DATA_OUT: now also J2.1 (Pin_1)
- net DIN: now also J2.9 (Pin_9)
- net GND: now also C_Polarized3.2, C_Polarized4.2, IC1.13 (DGND), C3.2, C6.2, C_Polarized12.2, J1.2, J1.3, J2.11 (Pin_11), U1.1 (GND), U2.1 (GND)
- net GUITAR_IN: now also J5.S, J5.SN
- net GUITAR_OUT: now also IC4.7 (VOUT_B), J4.S, J4.SN
- net LCH_IN: now also C_Polarized10.2, J3.5 (Pin_5); no longer C_Polarized6.2
- net LCH_OUT: now also J3.8 (Pin_8)
- net LRCLK: now also J2.3 (Pin_3)
- net MC/DEM0: now also J2.7 (Pin_7)
- net MC/DEM1: now also J2.8 (Pin_8)
- net ML/PDDA: now also J2.5 (Pin_5)
- net RCH_IN: now also IC4.1 (VOUT_A)
- net RCH_OUT: now also C_Polarized9.2; no longer C_Polarized10.2
- net RST/PDAD: now also J2.6 (Pin_6)
- net SYSCLK: now also J2.4 (Pin_4)
- net ZFLG: now also J2.10 (Pin_10), R1.1
- net at IC1.6 (VINL): now also C_Polarized10.1; no longer C_Polarized6.1
- net at C18.1, R10.2: now also IC4.6 (VIN_B-)
- net VGND: now reaches C25.1
- net VGND: now also IC5.6 (VIN_B-), IC5.7 (VOUT_B)
- net AGND: now reaches C25.2
- net AGND: now also C16.1, C17.1, C_Polarized1.2, C_Polarized2.2, C_Polarized6.2, C_Polarized7.2, C_Polarized8.2, IC1.22 (AGND2), IC1.23 (AGND1), C1.2, C2.2, C5.2, C7.2, C8.2, IC4.4 (VSS), IC5.3 (VINA+), IC5.4 (VSS), J3.3 (Pin_3), J4.T, J4.TN, J5.T, J5.TN, R17.2; no longer L2.1
- net VCC: now reaches L1.1
- net VCC: now also C_Polarized4.1, C3.1, D1.2 (A), U1.2 (VO), U2.3 (VI)
- net at IC1.20 (VOUTR): now also C_Polarized9.1; no longer C_Polarized10.1
- net at IC1.21 (VCOM): now also C_Polarized7.1; no longer C_Polarized9.1
- net at IC1.4 (VREF1): now also C_Polarized6.1; no longer C_Polarized7.1
- net at R14.2: now also IC4.3 (VINA+)
- net at C19.1, R11.2: now also IC4.2 (VINA-)
- net at R13.2: now also IC4.5 (VINB+)
- net +12V renamed VDD
- net VDD: now also L2.1, U2.2 (VO)
- net +3V3 renamed AVDD
- net AVDD: now also C1.1, C2.1, C6.1, C8.1, C_Polarized12.1, R1.2; no longer C_Polarized3.1, C_Polarized4.1
- net +5VD renamed AVCC
- net AVCC: now also C5.1, C7.1, IC4.8 (VDD), IC5.8 (VDD), R16.1
- removed net Earth: C16.1, C17.1, C_Polarized1.2, C_Polarized2.2, C_Polarized3.2, C_Polarized4.2, C_Polarized7.2, C_Polarized8.2, C_Polarized9.2, IC1.13 (DGND), IC1.22 (AGND2), IC1.23 (AGND1)
- new net: C_Polarized3.1, D1.1 (K), D2.1 (K), U1.3 (VI)
- new net: D2.2 (A), J1.1
- new net: IC5.1 (VOUT_A), IC5.2 (VINA-)
- new net VMID: IC5.5 (VINB+), R16.2, R17.1
- no-connect marks 0 -> 5
Other:
- note added: "AVCC = Analogue +5V"
- note added: "AVDD = Analogue +3.3V"
- note added: "Analogue part (1-7, 19-24 pins on Codec, upper part)"
- note added: "BW 56 Hz ... 32 kHz, 6 dB gain"
- note added: "CODEC - Datasheet pg. 33 circuit"
- note added: "Creating virtual ground VMID"
- note added: "Digital part (7-18 pins on Codec, lower part)"
- note added: "In and out pins"
- note added: "Input filtering (Multipple feedback Butterworth 20Hz...20kHz)"
- note added: "Input jack +12V to +5V and +3.3V (with analogue filtering)"
- note added: "Only mono"
- note added: "Output filtering"
- note added: "VCC = +3.3V"
- note added: "VCC = +5V"
- moved on the sheet: C11, C12, C16, C17, C18, C19, R10, R11, R13, R14, R3, R4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

Commit message: PCB v1.2
Connecting the digital and analogue ground. Analogue parts are put farther away from the digital parts, on the right side of the PCB.
Parts:
- removed J2: Conn_01x11_Pin, Connector_PinSocket_2.54mm:PinSocket_1x11_P2.54mm_Vertical, symbol Connector:Conn_01x11_Pin
- removed J3: Conn_01x08_Pin, Connector_PinSocket_2.54mm:PinSocket_1x08_P2.54mm_Vertical, symbol Connector:Conn_01x08_Pin
- removed U1: LD1117S12TR_SOT223, Package_TO_SOT_SMD:SOT-223-3_TabPin2, symbol Regulator_Linear:LD1117S12TR_SOT223
- added C10, C13, C22, C23, C24, C5, C9: 10u, Capacitor_SMD:C_1206_3216Metric, symbol Device:C
- added C_Polarized13: 870u, Capacitor_THT:CP_Radial_D4.0mm_P1.50mm, symbol Device:C_Polarized
- added J2: Conn_02x11_Odd_Even, Connector_PinHeader_2.54mm:PinHeader_2x11_P2.54mm_Vertical, symbol Connector_Generic:Conn_02x11_Odd_Even
- added J3: Conn_01x04_Pin, Connector_PinHeader_2.54mm:PinHeader_1x04_P2.54mm_Vertical, symbol Connector:Conn_01x04_Pin
- added U3: LD1117S50TR_SOT223, Package_TO_SOT_SMD:SOT-223-3_TabPin2, symbol Regulator_Linear:LD1117S50TR_SOT223
- C11, C12: value 1u -> 22u
- C16, C17: value 1.5n -> 10n
- C18, C19: value 560p -> 1n
- C21: renamed from C5; value 100n -> 10u; footprint Capacitor_SMD:C_0805_2012Metric -> Capacitor_SMD:C_1206_3216Metric
- R10, R11: value 2k -> 1.5k
- R6, R7: value 3.3k -> 1.5k
- R8, R9: value 1.6k -> 3k
- renumbered C25 to C20
Connections:
- net GND is gone; now on net AGND: C3.2, C4.2, C6.2, C_Polarized12.2, C_Polarized3.2, C_Polarized4.2, IC1.13 (DGND), J1.2, J1.3, U2.1 (GND)
- net AGND: now also C10.2, C13.2, C22.2, C23.2, C24.2, C5.2, C9.2, J2.1 (Pin_1), J2.11 (Pin_11), J2.13 (Pin_13), J2.15 (Pin_15), J2.17 (Pin_17), J2.19 (Pin_19), J2.21 (Pin_21), J2.22 (Pin_22), J2.3 (Pin_3), J2.5 (Pin_5), J2.7 (Pin_7), J2.9 (Pin_9), J3.4 (Pin_4), U3.1 (GND)
- net AVCC: now also C10.1, C9.1; no longer C21.1
- net AVDD: no longer C6.1, C_Polarized12.1, IC1.14 (VDD), R1.2
- net BIT: now also J2.4 (Pin_4)
- net DATA_OUT: now also J2.2 (Pin_2)
- net DIN: now also J2.18 (Pin_18)
- net GUITAR_OUT: now also C_Polarized13.2; no longer C18.2, IC4.7 (VOUT_B), R8.1
- net LCH_IN: now also J3.1 (Pin_1)
- net LCH_OUT: now also J3.3 (Pin_3)
- net LRCLK: now also J2.6 (Pin_6)
- net MC/DEM0: now also J2.14 (Pin_14)
- net MC/DEM1: now also J2.16 (Pin_16)
- net ML/PDDA: now also J2.10 (Pin_10)
- net RST/PDAD: now also J2.12 (Pin_12)
- net SYSCLK: now also J2.8 (Pin_8)
- net VCC: now also C21.1, C22.1, U3.2 (VO)
- net VDD: now also C6.1, C_Polarized12.1, IC1.14 (VDD), R1.2, C13.1, C23.1, C24.1, C5.1
- net ZFLG: now also J2.20 (Pin_20)
- net at C_Polarized3.1, D1.1 (K), D2.1 (K): now also U3.3 (VI)
- new net: C18.2, C_Polarized13.1, IC4.7 (VOUT_B), R8.1
- no-connect marks 5 -> 1
Other:
- note added: "BW 6 Hz ... 28 kHz, 6 dB gain"
- note added: "Decoupling for OPAMPs"
- note added: "Puffer capacitances for LDOs"
- note added: "Tie the GND and AGND"
- note removed: "BW 56 Hz ... 32 kHz, 6 dB gain"
- moved on the sheet: C21, J4, J5, R16, R17

Commit message: Forrasztáshoz
Parts:
- added D3: LED, LED_SMD:LED_0805_2012Metric_Pad1.15x1.40mm_HandSolder, symbol Device:LED
- added R2: 1k5, Resistor_SMD:R_0805_2012Metric_Pad1.20x1.40mm_HandSolder, symbol Device:R
- C13, C21, C22, C23, C24, C5: value 10u -> 150u
Connections:
- net AGND: now also R2.2
- net VCC: now also D3.2 (A)
- new net: D3.1 (K), R2.1
Other:
- moved on the sheet: C4, C_Polarized4, U2
